Commit message: updated xacro

File: src/herm_description/urdf/herm.urdf.xacro (robot description, xacro)
@@ -1,66 +1,96 @@
 <?xml version="1.0"?>
-<robot name="HERM" xmlns:xacro="http://www.ros.org/wiki/xacro">
-  <!-- ===================== -->
-  <!--  ROBOT PARAMETERS     -->
-  <!-- ===================== -->
-  <xacro:property name="base_radius" value="0.17"/>   <!-- 34cm diameter -->
-  <xacro:property name="base_height" value="0.05"/>   <!-- 5cm tall -->
-  <xacro:property name="wheel_radius" value="0.065"/> <!-- 6.5cm radius -->
-  <xacro:property name="wheel_width"  value="0.02"/>  <!-- 2cm thick -->
-  <xacro:property name="caster_radius" value="0.03"/> <!-- 3cm caster sphere -->
-  <!-- ===================== -->
-  <!--  GLOBAL MATERIALS     -->
+<robot name="herm" xmlns:xacro="http://www.ros.org/wiki/xacro">
+  <!-- ===================== -->
+  <!--    ROBOT PARAMETERS   -->
+  <!-- ===================== -->
+  <!-- Chassis dimensions (rectangular box) -->
+  <xacro:property name="chassis_length" value="0.40"/>
+  <xacro:property name="chassis_width" value="0.30"/>
+  <xacro:property name="chassis_height" value="0.08"/>
+  <!-- Wheel dimensions -->
+  <xacro:property name="wheel_radius" value="0.065"/>
+  <xacro:property name="wheel_width" value="0.04"/>
+  <!-- Wheel positions -->
+  <xacro:property name="wheelbase" value="0.30"/>
+  <xacro:property name="track_width" value="0.34"/>
+  <!-- Layer/Plate dimensions -->
+  <xacro:property name="plate_length" value="0.35"/>
+  <xacro:property name="plate_width" value="0.25"/>
+  <xacro:property name="plate_thickness" value="0.005"/>
+  <!-- Standoff dimensions -->
+  <xacro:property name="standoff_radius" value="0.006"/>
+  <xacro:property name="standoff_height_1" value="0.07"/>
+  <xacro:property name="standoff_height_2" value="0.06"/>
+  <xacro:property name="standoff_height_3" value="0.06"/>
+  <!-- LiDAR dimensions -->
+  <xacro:property name="lidar_radius" value="0.04"/>
+  <xacro:property name="lidar_height" value="0.05"/>
+  <!-- Camera dimensions -->
+  <xacro:property name="camera_size" value="0.04"/>
+  <!-- ===================== -->
+  <!--       MATERIALS       -->
   <!-- ===================== -->
   <material name="black">
-    <color rgba="0.0 0.0 0.0 1.0"/>
-  </material>
-  <material name="gray">
-    <color rgba="0.5 0.5 0.5 1.0"/>
+    <color rgba="0.1 0.1 0.1 1.0"/>
+  </material>
+  <material name="dark_gray">
+    <color rgba="0.2 0.2 0.2 1.0"/>
+  </material>
+  <material name="light_gray">
+    <color rgba="0.7 0.7 0.7 1.0"/>
   </material>
   <material name="blue">
-    <color rgba="0.1 0.2 1.0 1.0"/>
+    <color rgba="0.0 0.2 0.8 1.0"/>
   </material>
   <material name="red">
-    <color rgba="1.0 0.0 0.0 1.0"/>
-  </material>
-  <!-- ===================== -->
-  <!--      BASE LINK        -->
-  <!-- ===================== -->
-  <!-- Turtlebot-style round base -->
+    <color rgba="0.8 0.0 0.0 1.0"/>
+  </material>
+  <material name="silver">
+    <color rgba="0.75 0.75 0.75 1.0"/>
+  </material>
+  <!-- ===================== -->
+  <!--     BASE FOOTPRINT    -->
+  <!-- ===================== -->
+  <link name="base_footprint"/>
+  <!-- ===================== -->
+  <!--       BASE LINK       -->
+  <!-- ===================== -->
   <link name="base_link">
     <visual>
       <geometry>
-        <cylinder radius="${base_radius}" length="${base_height}"/>
-      </geometry>
-      <origin xyz="0 0 0" rpy="0 0 0"/>
-      <material name="gray"/>
-    </visual>
-    <collision>
-      <geometry>
-        <cylinder radius="${base_radius}" length="${base_height}"/>
-      </geometry>
-      <origin xyz="0 0 0" rpy="0 0 0"/>
-    </collision>
-    <inertial>
-      <mass value="6.0"/>
-      <origin xyz="0 0 0" rpy="0 0 0"/>
-      <inertia
-        ixx="0.15" ixy="0.0" ixz="0.0"
-        iyy="0.15" iyz="0.0"
-        izz="0.20"/>
-    </inertial>
-  </link>
-  <!-- ===================== -->
-  <!--    2WD DRIVE WHEELS   -->
-  <!-- ===================== -->
-  <!-- Wheel macro -->
-  <xacro:macro name="drive_wheel" params="name y">
-    <link name="${name}">
+        <box size="${chassis_length} ${chassis_width} ${chassis_height}"/>
+      </geometry>
+      <origin xyz="0 0 0" rpy="0 0 0"/>
+      <material name="dark_gray"/>
+    </visual>
+    <collision>
+      <geometry>
+        <box size="${chassis_length} ${chassis_width} ${chassis_height}"/>
+      </geometry>
+      <origin xyz="0 0 0" rpy="0 0 0"/>
+    </collision>
+    <inertial>
+      <mass value="8.0"/>
+      <origin xyz="0 0 0" rpy="0 0 0"/>
+      <inertia ixx="0.1" ixy="0.0" ixz="0.0"
+               iyy="0.15" iyz="0.0"
+               izz="0.2"/>
+    </inertial>
+  </link>
+  <joint name="base_joint" type="fixed">
+    <parent link="base_footprint"/>
+    <child link="base_link"/>
+    <origin xyz="0 0 ${wheel_radius + chassis_height/2}" rpy="0 0 0"/>
+  </joint>
+  <!-- ===================== -->
+  <!--      WHEEL MACRO      -->
+  <!-- ===================== -->
+  <xacro:macro name="wheel" params="prefix x_offset y_offset">
+    <link name="${prefix}_wheel_link">
       <visual>
         <geometry>
           <cylinder radius="${wheel_radius}" length="${wheel_width}"/>
         </geometry>
-        <!-- Rotate so cylinder axis is along robot x -->
-        <origin xyz="0 0 0" rpy="0 1.5707 0"/>
+        <origin xyz="0 0 0" rpy="${pi/2} 0 0"/>
         <material name="black"/>
       </visual>
@@ -69,41 +99,245 @@
           <cylinder radius="${wheel_radius}" length="${wheel_width}"/>
         </geometry>
-        <origin xyz="0 0 0" rpy="0 1.5707 0"/>
+        <origin xyz="0 0 0" rpy="${pi/2} 0 0"/>
       </collision>
       <inertial>
-        <mass value="0.3"/>
-        <origin xyz="0 0 0" rpy="0 0 0"/>
-        <inertia
-          ixx="0.002" ixy="0.0" ixz="0.0"
-          iyy="0.002" iyz="0.0"
-          izz="0.002"/>
+        <mass value="0.5"/>
+        <origin xyz="0 0 0" rpy="${pi/2} 0 0"/>
+        <inertia ixx="0.001" ixy="0.0" ixz="0.0"
+                 iyy="0.001" iyz="0.0"
+                 izz="0.0015"/>
       </inertial>
     </link>
-    <!-- Continuous joint for differential drive -->
-    <joint name="${name}_joint" type="continuous">
+    <joint name="${prefix}_wheel_joint" type="continuous">
       <parent link="base_link"/>
-      <child link="${name}"/>
-      <!-- Place wheel on side at base radius, slightly below base -->
-      <origin xyz="0 ${y} -${base_height/2}" rpy="0 0 0"/>
+      <child link="${prefix}_wheel_link"/>
+      <origin xyz="${x_offset} ${y_offset} ${-chassis_height/2}" rpy="0 0 0"/>
       <axis xyz="0 1 0"/>
+      <dynamics damping="0.1" friction="0.5"/>
     </joint>
   </xacro:macro>
-  <!-- Left and right wheels -->
-  <xacro:drive_wheel name="left_wheel"  y="${ base_radius}"/>
-  <xacro:drive_wheel name="right_wheel" y="-${base_radius}"/>
-  <!-- ===================== -->
-  <!--      CASTER WHEEL     -->
-  <!-- ===================== -->
-  <link name="caster_wheel">
-    <visual>
-      <geometry>
-        <sphere radius="${caster_radius}"/>
-      </geometry>
-      <origin xyz="0 0 0" rpy="0 0 0"/>
-      <material name="black"/>
-    </visual>
-    <collision>
-      <geometry>
-        <sphere radius="${caster_radius}"/>
+  <!-- Four wheels (skid-steer 4WD) -->
+  <xacro:wheel prefix="front_left"  x_offset="${wheelbase/2}"  y_offset="${track_width/2}"/>
+  <xacro:wheel prefix="front_right" x_offset="${wheelbase/2}"  y_offset="${-track_width/2}"/>
+  <xacro:wheel prefix="rear_left"   x_offset="${-wheelbase/2}" y_offset="${track_width/2}"/>
+  <xacro:wheel prefix="rear_right"  x_offset="${-wheelbase/2}" y_offset="${-track_width/2}"/>
+  <!-- ===================== -->
+  <!--    STANDOFF MACRO     -->
+  <!-- ===================== -->
+  <xacro:macro name="standoff" params="prefix parent x_offset y_offset z_offset height">
+    <link name="${prefix}_standoff_link">
+      <visual>
+        <geometry>
+          <cylinder radius="${standoff_radius}" length="${height}"/>
+        </geometry>
+        <origin xyz="0 0 0" rpy="0 0 0"/>
+        <material name="silver"/>
+      </visual>
+      <collision>
+        <geometry>
+          <cylinder radius="${standoff_radius}" length="${height}"/>
+        </geometry>
+        <origin xyz="0 0 0" rpy="0 0 0"/>
+      </collision>
+      <inertial>
+        <mass value="0.02"/>
+        <origin xyz="0 0 0" rpy="0 0 0"/>
+        <inertia ixx="0.00001" ixy="0.0" ixz="0.0"
+                 iyy="0.00001" iyz="0.0"
+                 izz="0.000001"/>
+      </inertial>
+    </link>
+    <joint name="${prefix}_standoff_joint" type="fixed">
+      <parent link="${parent}"/>
+      <child link="${prefix}_standoff_link"/>
+      <origin xyz="${x_offset} ${y_offset} ${z_offset}" rpy="0 0 0"/>
+    </joint>
+  </xacro:macro>
+  <!-- ===================== -->
+  <!--   LAYER 1 (MIDDLE)    -->
+  <!-- ===================== -->
+  <!-- Standoffs from base to layer 1 -->
+  <xacro:property name="standoff_x" value="${plate_length/2 - 0.02}"/>
+  <xacro:property name="standoff_y" value="${plate_width/2 - 0.02}"/>
+  <xacro:standoff prefix="layer1_fl" parent="base_link"
+                  x_offset="${standoff_x}" y_offset="${standoff_y}"
+                  z_offset="${chassis_height/2 + standoff_height_1/2}" height="${standoff_height_1}"/>
+  <xacro:standoff prefix="layer1_fr" parent="base_link"
+                  x_offset="${standoff_x}" y_offset="${-standoff_y}"
+                  z_offset="${chassis_height/2 + standoff_height_1/2}" height="${standoff_height_1}"/>
+  <xacro:standoff prefix="layer1_rl" parent="base_link"
+                  x_offset="${-standoff_x}" y_offset="${standoff_y}"
+                  z_offset="${chassis_height/2 + standoff_height_1/2}" height="${standoff_height_1}"/>
+  <xacro:standoff prefix="layer1_rr" parent="base_link"
+                  x_offset="${-standoff_x}" y_offset="${-standoff_y}"
+                  z_offset="${chassis_height/2 + standoff_height_1/2}" height="${standoff_height_1}"/>
+  <!-- Layer 1 plate -->
+  <link name="layer1_link">
+    <visual>
+      <geometry>
+        <box size="${plate_length} ${plate_width} ${plate_thickness}"/>
+      </geometry>
+      <origin xyz="0 0 0" rpy="0 0 0"/>
+      <material name="light_gray"/>
+    </visual>
+    <collision>
+      <geometry>
+        <box size="${plate_length} ${plate_width} ${plate_thickness}"/>
+      </geometry>
+      <origin xyz="0 0 0" rpy="0 0 0"/>
+    </collision>
+    <inertial>
+      <mass value="0.3"/>
+      <origin xyz="0 0 0" rpy="0 0 0"/>
+      <inertia ixx="0.002" ixy="0.0" ixz="0.0"
+               iyy="0.001" iyz="0.0"
+               izz="0.003"/>
+    </inertial>
+  </link>
+  <joint name="layer1_joint" type="fixed">
+    <parent link="base_link"/>
+    <child link="layer1_link"/>
+    <origin xyz="0 0 ${chassis_height/2 + standoff_height_1 + plate_thickness/2}" rpy="0 0 0"/>
+  </joint>
+  <!-- ===================== -->
+  <!--   LAYER 2 (MIDDLE)    -->
+  <!-- ===================== -->
+  <!-- Standoffs from layer 1 to layer 2 -->
+  <xacro:standoff prefix="layer2_fl" parent="layer1_link"
+                  x_offset="${standoff_x}" y_offset="${standoff_y}"
+                  z_offset="${plate_thickness/2 + standoff_height_2/2}" height="${standoff_height_2}"/>
+  <xacro:standoff prefix="layer2_fr" parent="layer1_link"
+                  x_offset="${standoff_x}" y_offset="${-standoff_y}"
+                  z_offset="${plate_thickness/2 + standoff_height_2/2}" height="${standoff_height_2}"/>
+  <xacro:standoff prefix="layer2_rl" parent="layer1_link"
+                  x_offset="${-standoff_x}" y_offset="${standoff_y}"
+                  z_offset="${plate_thickness/2 + standoff_height_2/2}" height="${standoff_height_2}"/>
+  <xacro:standoff prefix="layer2_rr" parent="layer1_link"
+                  x_offset="${-standoff_x}" y_offset="${-standoff_y}"
+                  z_offset="${plate_thickness/2 + standoff_height_2/2}" height="${standoff_height_2}"/>
+  <!-- Layer 2 plate (middle) -->
+  <link name="layer2_link">
+    <visual>
+      <geometry>
+        <box size="${plate_length} ${plate_width} ${plate_thickness}"/>
+      </geometry>
+      <origin xyz="0 0 0" rpy="0 0 0"/>
+      <material name="light_gray"/>
+    </visual>
+    <collision>
+      <geometry>
+        <box size="${plate_length} ${plate_width} ${plate_thickness}"/>
+      </geometry>
+      <origin xyz="0 0 0" rpy="0 0 0"/>
+    </collision>
+    <inertial>
+      <mass value="0.3"/>
+      <origin xyz="0 0 0" rpy="0 0 0"/>
+      <inertia ixx="0.002" ixy="0.0" ixz="0.0"
+               iyy="0.001" iyz="0.0"
+               izz="0.003"/>
+    </inertial>
+  </link>
+  <joint name="layer2_joint" type="fixed">
+    <parent link="layer1_link"/>
+    <child link="layer2_link"/>
+    <origin xyz="0 0 ${plate_thickness/2 + standoff_height_2 + plate_thickness/2}" rpy="0 0 0"/>
+  </joint>
+  <!-- ===================== -->
+  <!--    LAYER 3 (TOP)      -->
+  <!-- ===================== -->
+  <!-- Standoffs from layer 2 to layer 3 -->
+  <xacro:standoff prefix="layer3_fl" parent="layer2_link"
+                  x_offset="${standoff_x}" y_offset="${standoff_y}"
+                  z_offset="${plate_thickness/2 + standoff_height_3/2}" height="${standoff_height_3}"/>
+  <xacro:standoff prefix="layer3_fr" parent="layer2_link"
+                  x_offset="${standoff_x}" y_offset="${-standoff_y}"
+                  z_offset="${plate_thickness/2 + standoff_height_3/2}" height="${standoff_height_3}"/>
+  <xacro:standoff prefix="layer3_rl" parent="layer2_link"
+                  x_offset="${-standoff_x}" y_offset="${standoff_y}"
+                  z_offset="${plate_thickness/2 + standoff_height_3/2}" height="${standoff_height_3}"/>
+  <xacro:standoff prefix="layer3_rr" parent="layer2_link"
+                  x_offset="${-standoff_x}" y_offset="${-standoff_y}"
+                  z_offset="${plate_thickness/2 + standoff_height_3/2}" height="${standoff_height_3}"/>
+  <!-- Layer 3 plate (top) -->
+  <link name="layer3_link">
+    <visual>
+      <geometry>
+        <box size="${plate_length} ${plate_width} ${plate_thickness}"/>
+      </geometry>
+      <origin xyz="0 0 0" rpy="0 0 0"/>
+      <material name="light_gray"/>
+    </visual>
+    <collision>
+      <geometry>
+        <box size="${plate_length} ${plate_width} ${plate_thickness}"/>
+      </geometry>
+      <origin xyz="0 0 0" rpy="0 0 0"/>
+    </collision>
+    <inertial>
+      <mass value="0.3"/>
+      <origin xyz="0 0 0" rpy="0 0 0"/>
+      <inertia ixx="0.002" ixy="0.0" ixz="0.0"
+               iyy="0.001" iyz="0.0"
+               izz="0.003"/>
+    </inertial>
+  </link>
+  <joint name="layer3_joint" type="fixed">
+    <parent link="layer2_link"/>
+    <child link="layer3_link"/>
+    <origin xyz="0 0 ${plate_thickness/2 + standoff_height_3 + plate_thickness/2}" rpy="0 0 0"/>
+  </joint>
+  <!-- ===================== -->
+  <!--  CAMERA (on Layer 2)  -->
+  <!-- ===================== -->
+  <link name="camera_link">
+    <visual>
+      <geometry>
+        <box size="${camera_size} ${camera_size} ${camera_size * 1.5}"/>
+      </geometry>
+      <origin xyz="0 0 0" rpy="0 0 0"/>
+      <material name="blue"/>
+    </visual>
+    <collision>
+      <geometry>
+        <box size="${camera_size} ${camera_size} ${camera_size * 1.5}"/>
+      </geometry>
+      <origin xyz="0 0 0" rpy="0 0 0"/>
+    </collision>
+    <inertial>
+      <mass value="0.15"/>
+      <origin xyz="0 0 0" rpy="0 0 0"/>
+      <inertia ixx="0.00005" ixy="0.0" ixz="0.0"
+               iyy="0.00005" iyz="0.0"
+               izz="0.00003"/>
+    </inertial>
+  </link>
+  <!-- Camera positioned towards front on layer 2 -->
+  <joint name="camera_joint" type="fixed">
+    <parent link="layer2_link"/>
+    <child link="camera_link"/>
+    <origin xyz="${plate_length/2 - camera_size} 0 ${plate_thickness/2 + camera_size * 0.75}" rpy="0 0 0"/>
+  </joint>
+  <!-- Camera optical frame (Z forward, X right, Y down per REP-103) -->
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