Commit message: update for ros gz harmonic

File: src/herm_simulation/urdf/herm_gazebo.urdf.xacro (robot description, xacro)
@@ -6,61 +6,49 @@
   <!--   GAZEBO PROPERTIES   -->
   <!-- ===================== -->
-  <!-- Base link -->
+  <!-- Base link friction -->
   <gazebo reference="base_link">
-    <material>Gazebo/Grey</material>
-  </gazebo>
-  <!-- Layer plates -->
-  <gazebo reference="layer1_link">
-    <material>Gazebo/White</material>
-  </gazebo>
-  <gazebo reference="layer2_link">
-    <material>Gazebo/White</material>
-  </gazebo>
-  <gazebo reference="layer3_link">
-    <material>Gazebo/White</material>
-  </gazebo>
-  <!-- Wheels -->
-  <gazebo reference="front_left_wheel_link">
-    <material>Gazebo/Black</material>
-    <mu1>1.0</mu1>
-    <mu2>1.0</mu2>
-    <kp>1000000.0</kp>
-    <kd>100.0</kd>
-  </gazebo>
-  <gazebo reference="front_right_wheel_link">
-    <material>Gazebo/Black</material>
-    <mu1>1.0</mu1>
-    <mu2>1.0</mu2>
-    <kp>1000000.0</kp>
-    <kd>100.0</kd>
-  </gazebo>
-  <gazebo reference="rear_left_wheel_link">
-    <material>Gazebo/Black</material>
-    <mu1>1.0</mu1>
-    <mu2>1.0</mu2>
-    <kp>1000000.0</kp>
-    <kd>100.0</kd>
-  </gazebo>
-  <gazebo reference="rear_right_wheel_link">
-    <material>Gazebo/Black</material>
-    <mu1>1.0</mu1>
-    <mu2>1.0</mu2>
-    <kp>1000000.0</kp>
-    <kd>100.0</kd>
-  </gazebo>
-  <!-- LiDAR -->
-  <gazebo reference="base_scan">
-    <material>Gazebo/Red</material>
-  </gazebo>
-  <!-- Camera -->
-  <gazebo reference="camera_link">
-    <material>Gazebo/Blue</material>
-  </gazebo>
-  <!-- ===================== -->
-  <!--  DIFF DRIVE PLUGIN    -->
-  <!-- ===================== -->
+    <collision>
+      <surface>
+        <friction>
+          <ode>
+            <mu>0.5</mu>
+            <mu2>0.5</mu2>
+          </ode>
+        </friction>
+      </surface>
+    </collision>
+  </gazebo>
+  <!-- Wheel friction properties -->
+  <xacro:macro name="wheel_gazebo" params="wheel_name">
+    <gazebo reference="${wheel_name}_link">
+      <collision>
+        <surface>
+          <friction>
+            <ode>
+              <mu>1.0</mu>
+              <mu2>1.0</mu2>
+              <fdir1>0 0 1</fdir1>
+            </ode>
+          </friction>
+          <contact>
+            <ode>
+              <kp>1000000.0</kp>
+              <kd>100.0</kd>
+            </ode>
+          </contact>
+        </surface>
+      </collision>
+    </gazebo>
+  </xacro:macro>
+  <xacro:wheel_gazebo wheel_name="front_left_wheel"/>
+  <xacro:wheel_gazebo wheel_name="front_right_wheel"/>
+  <xacro:wheel_gazebo wheel_name="rear_left_wheel"/>
+  <xacro:wheel_gazebo wheel_name="rear_right_wheel"/>
+  <!-- ===================================== -->
+  <!--  GAZEBO HARMONIC DIFF DRIVE PLUGIN    -->
+  <!-- ===================================== -->
   <gazebo>
-    <plugin name="diff_drive_controller" filename="libgazebo_ros_diff_drive.so">
-      <!-- Wheel joints -->
+    <plugin filename="gz-sim-diff-drive-system" name="gz::sim::systems::DiffDrive">
+      <!-- Wheel joints (4WD skid-steer) -->
       <left_joint>front_left_wheel_joint</left_joint>
       <left_joint>rear_left_wheel_joint</left_joint>
@@ -69,28 +57,36 @@
       <!-- Kinematics -->
       <wheel_separation>0.34</wheel_separation>
-      <wheel_diameter>0.13</wheel_diameter>
+      <wheel_radius>0.065</wheel_radius>
       <!-- Limits -->
-      <max_wheel_torque>20</max_wheel_torque>
-      <max_wheel_acceleration>1.0</max_wheel_acceleration>
-      <!-- Output -->
-      <publish_odom>true</publish_odom>
-      <publish_odom_tf>true</publish_odom_tf>
-      <publish_wheel_tf>true</publish_wheel_tf>
-      <odometry_frame>odom</odometry_frame>
+      <max_linear_acceleration>1.0</max_linear_acceleration>
+      <max_angular_acceleration>2.0</max_angular_acceleration>
+      <!-- TF frames -->
+      <odom_frame>odom</odom_frame>
       <robot_base_frame>base_footprint</robot_base_frame>
-      <!-- Topic names -->
-      <command_topic>cmd_vel</command_topic>
-      <odometry_topic>odom</odometry_topic>
+      <!-- Topic names (Gazebo topics, bridged to ROS2) -->
+      <topic>cmd_vel</topic>
+      <odom_topic>odom</odom_topic>
+      <tf_topic>tf</tf_topic>
+      <!-- Publish odometry -->
+      <odom_publish_frequency>50</odom_publish_frequency>
     </plugin>
-  </gazebo>
-  <!-- ===================== -->
-  <!--    LIDAR PLUGIN       -->
-  <!-- ===================== -->
+    <!-- Joint state publisher -->
+    <plugin filename="gz-sim-joint-state-publisher-system" name="gz::sim::systems::JointStatePublisher">
+      <topic>joint_states</topic>
+      <joint_name>front_left_wheel_joint</joint_name>
+      <joint_name>front_right_wheel_joint</joint_name>
+      <joint_name>rear_left_wheel_joint</joint_name>
+      <joint_name>rear_right_wheel_joint</joint_name>
+    </plugin>
+  </gazebo>
+  <!-- ===================================== -->
+  <!--    LIDAR SENSOR (GPU LIDAR)           -->
+  <!-- ===================================== -->
   <gazebo reference="base_scan">
-    <sensor type="ray" name="rplidar_sensor">
+    <sensor name="lidar" type="gpu_lidar">
       <pose>0 0 0 0 0 0</pose>
-      <visualize>true</visualize>
+      <topic>scan</topic>
       <update_rate>10</update_rate>
-      <ray>
+      <lidar>
         <scan>
           <horizontal>
@@ -100,4 +96,10 @@
             <max_angle>3.14159</max_angle>
           </horizontal>
+          <vertical>
+            <samples>1</samples>
+            <resolution>1</resolution>
+            <min_angle>0</min_angle>
+            <max_angle>0</max_angle>
+          </vertical>
         </scan>
         <range>
@@ -111,21 +113,18 @@
           <stddev>0.01</stddev>
         </noise>
-      </ray>
-      <plugin name="gazebo_ros_rplidar" filename="libgazebo_ros_ray_sensor.so">
-        <ros>
-          <remapping>~/out:=scan</remapping>
-        </ros>
-        <output_type>sensor_msgs/LaserScan</output_type>
-        <frame_name>base_scan</frame_name>
-      </plugin>
+      </lidar>
+      <always_on>true</always_on>
+      <visualize>true</visualize>
     </sensor>
   </gazebo>
-  <!-- ===================== -->
-  <!--    CAMERA PLUGIN      -->
-  <!-- ===================== -->
+  <!-- ===================================== -->
+  <!--    CAMERA SENSOR                      -->
+  <!-- ===================================== -->
   <gazebo reference="camera_link">
-    <sensor type="camera" name="insta360_camera">
-      <update_rate>30.0</update_rate>
-      <camera name="camera">
+    <sensor name="camera" type="camera">
+      <pose>0 0 0 0 0 0</pose>
+      <topic>camera/image_raw</topic>
+      <update_rate>30</update_rate>
+      <camera>
         <horizontal_fov>1.3962634</horizontal_fov>
         <image>
@@ -144,20 +143,18 @@
         </noise>
       </camera>
-      <plugin name="gazebo_ros_camera" filename="libgazebo_ros_camera.so">
-        <ros>
-          <remapping>~/image_raw:=camera/image_raw</remapping>
-          <remapping>~/camera_info:=camera/camera_info</remapping>
-        </ros>
-        <camera_name>camera</camera_name>
-        <frame_name>camera_optical_frame</frame_name>
-      </plugin>
+      <always_on>true</always_on>
+      <visualize>true</visualize>
     </sensor>
   </gazebo>
-  <!-- ===================== -->
-  <!--      IMU PLUGIN       -->
-  <!-- ===================== -->
+  <!-- Camera optical frame -->
+  <gazebo reference="camera_optical_frame">
+  </gazebo>
+  <!-- ===================================== -->
+  <!--      IMU SENSOR                       -->
+  <!-- ===================================== -->
   <gazebo reference="imu_link">
-    <sensor type="imu" name="imu_sensor">
-      <always_on>true</always_on>
+    <sensor name="imu" type="imu">
+      <pose>0 0 0 0 0 0</pose>
+      <topic>imu/data</topic>
       <update_rate>100</update_rate>
       <imu>
@@ -203,10 +200,5 @@
         </linear_acceleration>
       </imu>
-      <plugin name="gazebo_ros_imu" filename="libgazebo_ros_imu_sensor.so">
-        <ros>
-          <remapping>~/out:=imu/data</remapping>
-        </ros>
-        <frame_name>imu_link</frame_name>
-      </plugin>
+      <always_on>true</always_on>
     </sensor>
   </gazebo>
